File: larson_vu/larson_vu/larson_vu.kicad_sch (KiCad schematic)
At the start: 0 parts

Commit message: Added larson scanner PCB
Parts:
- added A1, A2: SJ1-3533NG, symbol SJ1-3533NG:SJ1-3533NG
- added C1, C3, C5, C7: (no value), symbol Device:C_Small
- added C2, C8: 0.1uF, Capacitor_THT:C_Disc_D5.0mm_W2.5mm_P2.50mm, symbol Device:C_Small
- added C4: 1nF, Capacitor_THT:C_Disc_D5.0mm_W2.5mm_P2.50mm, symbol Device:C_Small
- added C6: 33pF, Capacitor_THT:C_Disc_D5.0mm_W2.5mm_P2.50mm, symbol Device:C_Small
- added C9: (no value), symbol Device:C_Polarized
- added H1: (no value), symbol Mechanical:MountingHole_Pad
- added H2, H3, H4: MountHole, MountingHole:MountingHole_3.2mm_M3_Pad, symbol Mechanical:MountingHole_Pad
- added J1, J2: (no value), symbol Connector_Generic:Conn_01x02
- added J3: (no value), symbol Connector_Generic:Conn_01x04
- added R1, R3: (no value), symbol Device:R
- added R2: 22k, Resistor_THT:R_Axial_DIN0207_L6.3mm_D2.5mm_P7.62mm_Horizontal, symbol Device:R
- added R4: 200k, Resistor_THT:R_Axial_DIN0207_L6.3mm_D2.5mm_P7.62mm_Horizontal, symbol Device:R
- added U1: (no value), symbol teensy:Teensy3.2
- added U2: (no value), symbol Audio:MSGEQ7
- added U3: MSGEQ7, Package_DIP:DIP-8_W7.62mm_Socket, symbol Audio:MSGEQ7
Connections:
- new net: C5.1, R3.2, U2.8 (CKIN)
- new net: C4.1, R2.2
- new net: C3.1, R1.2
- new net: C3.2, U2.5 (IN)
- new net: C8.2, U3.6 (GND)
- new net: C7.2, U2.6 (GND)
- new net: C6.1, R4.2, U3.8 (CKIN)
- new net: C4.2, U3.5 (IN)
- new net +5V: C1.2, C2.2, C9.1, J1.2 (Pin_2), J3.4 (Pin_4), R3.1, R4.1, U1.33 (Vin), U2.1 (VDD), U3.1 (VDD)
- new net A0: U1.21 (14_A0_SCK), U2.3 (OUT)
- new net A1: U1.22 (15_A1_CS_Touch), U3.3 (OUT)
- new net AUDIO_L: A1.2, A2.2, R1.1
- new net AUDIO_R: A1.3, A2.3, R2.1
- new net GND: A1.1, A2.1, C1.1, C2.1, C5.2, C6.2, C7.1, C8.1, C9.2, H1.1, H2.1, H3.1, H4.1, J1.1 (Pin_1), J2.1 (Pin_1), J3.1 (Pin_1), U1.1 (GND), U1.17 (GND), U1.32 (AGND), U1.53 (GND), U2.2 (VSS), U3.2 (VSS)
- new net LED_CLOCK: J3.3 (Pin_3), U1.20 (13_LED_SCK)
- new net LED_DATA: J3.2 (Pin_2), U1.13 (11_DOUT)
- new net RESET: U1.24 (17_A3_SDA0_Touch), U2.7 (RESET), U3.7 (RESET)
- new net RX: J2.2 (Pin_2), U1.2 (0_RX1_Touch)
- new net STROBE: U1.23 (16_A2_SCL0_Touch), U2.4 (STROBE), U3.4 (STROBE)
